File: testCoupon.kicad_pcb (KiCad board)
At the start: 4 copper layers, 41.8 x 57 mm, 13 parts, among them J1 Conn_Coaxial, J10 Conn_Coaxial, J2 Conn_Coaxial, J3 Conn_Coaxial, J4 Conn_Coaxial, J5 Conn_Coaxial, J6 Conn_Coaxial, J7 Conn_Coaxial, J8 Conn_Coaxial, J9 Conn_Coaxial

Commit message: fab files
Other:
- board text added: "JLCJLCJLCJLC"
Changed lines of the file:
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@@
       (layerselection 0x00010fc_ffffffff)
       (disableapertmacros false)
-      (usegerberextensions false)
+      (usegerberextensions true)
       (usegerberattributes true)
       (usegerberadvancedattributes true)
-      (creategerberjobfile true)
+      (creategerberjobfile false)
       (svguseinch false)
       (svgprecision 6)
@@
       (psa4output false)
       (plotreference true)
-      (plotvalue true)
+      (plotvalue false)
       (plotinvisibletext false)
       (sketchpadsonfab false)
-      (subtractmaskfromsilk false)
+      (subtractmaskfromsilk true)
       (outputformat 1)
       (mirror false)
-      (drillshape 1)
+      (drillshape 0)
       (scaleselection 1)
-      (outputdirectory "")
+      (outputdirectory "gerber/")
     )
   )
@@
   (gr_rect (start 140.75 92.9) (end 136.05 95.3) (layer "F.Mask") (width 0.15) (fill solid))
   (gr_rect (start 135.3 114.6) (end 177.1 57.6) (layer "Edge.Cuts") (width 0.1) (fill none))
+  (gr_text "JLCJLCJLCJLC" (at 156.8 59.2) (layer "B.SilkS")
+    (effects (font (size 1 1) (thickness 0.15)) (justify mirror))
+  )
   (gr_text "JLCPCB Microstrip" (at 155.4 66.5) (layer "F.SilkS")
     (effects (font (size 1 1) (thickness 0.15)))
   )
-  (gr_text "Saturn PCB Coplanar Waveguide" (at 157 101.3) (layer "F.SilkS")
+  (gr_text "Saturn PCB Coplanar Waveguide" (at 156.5 101.3) (layer "F.SilkS")
     (effects (font (size 1 1) (thickness 0.15)))
   )
@@
     (effects (font (size 1 1) (thickness 0.15)))
   )
-  (gr_text "Sonnet Optimized Coplanar Waveguide" (at 157 112.9) (layer "F.SilkS")
+  (gr_text "Sonnet Optimized Coplanar Waveguide" (at 156.5 112.9) (layer "F.SilkS")
     (effects (font (size 1 1) (thickness 0.15)))
   )

Commit message: why me
whyyyyyy
whyyyyyyyyyyyyyyyyy
whyyyyyyyyyyyyyyyyyyyyyyyyyyy
Routing:
- net GND: vias 104 -> 96
Other:
- board size 41.8 x 57 mm -> 40.5 x 57 mm
